Commit message: 将livox驱动的配置替换为robosense

File: My_nav/src/gazebo/pb_rm_simulation/urdf/simulation_waking_robot.xacro (robot description, xacro)
@@ -11,5 +11,5 @@
     </inertial>
   </xacro:macro>
-  <!-- base_link to livox_frame -->
+  <!-- base_link to rslidar (legacy frame: livox_frame) -->
   <xacro:arg name="xyz" default="0.12 0.0 0.175" />
   <xacro:arg name="rpy" default="0 0 0" />
@@ -182,5 +182,5 @@
     <material>Gazebo/BuildingFrame</material>
   </gazebo>
-  <gazebo reference="livox_frame">
+  <gazebo reference="rslidar">
     <material>Gazebo/LightBlueLaser</material>
   </gazebo>
@@ -212,8 +212,8 @@
     </plugin>
   </gazebo>
-  <!-- mid360_imu plugin -->
+  <!-- Airy Lite IMU simulation -->
   <!-- https://github.com/ros-simulation/gazebo_ros_pkgs/wiki/ROS-2-Migration:-IMU-Sensors -->
   <gazebo reference="imu_link">
-    <sensor name="mid360_imu" type="imu">
+    <sensor name="airy_lite_imu" type="imu">
       <always_on>true</always_on>
       <update_rate>100</update_rate>
@@ -221,5 +221,6 @@
         <ros>
           <namespace>/</namespace>
-          <remapping>~/out:=/livox/imu</remapping>
+          <!-- Livox: ~/out:=/livox/imu -->
+          <remapping>~/out:=/rslidar_imu_data</remapping>
         </ros>
         <frame_name>imu_link</frame_name>
@@ -227,8 +228,8 @@
     </sensor>
   </gazebo>
-  <!-- Livox-Mid360  -->
-  <xacro:include filename="$(find ros2_livox_simulation)/urdf/mid360.xacro" />
-  <xacro:mid360 name="livox_frame" parent="base_link" topic="/livox/lidar">
+  <!-- Legacy Livox include/macro: ros2_livox_simulation, xacro:mid360 -->
+  <xacro:include filename="$(find robosense_sim_ros2)/urdf/airy_lite.xacro" />
+  <xacro:airy_lite name="rslidar" parent="base_link" topic="/rslidar_points">
     <origin xyz="$(arg xyz)" rpy="$(arg rpy)" />
-  </xacro:mid360>
+  </xacro:airy_lite>
 </robot>

File: My_nav/src/rm_nav_bringup/urdf/sentry_robot_real.xacro (robot description, xacro)
@@ -11,5 +11,5 @@
     </inertial>
   </xacro:macro>
-  <!-- base_link to livox_frame -->
+  <!-- base_link to Airy Lite rslidar frame (legacy name: livox_frame) -->
   <xacro:arg name="xyz" default="0.0 0.045 0.49" />
   <xacro:arg name="rpy" default="0 0 0" />
@@ -128,6 +128,6 @@
     <origin rpy="${-PI/2} 0 0" xyz="-0.1 -0.13 0"/>
   </joint>
-  <!-- Livox-Mid360  -->
-  <link name="livox_frame">
+  <!-- Legacy Livox frame name: livox_frame. Airy Lite frame follows rslidar_sdk/config/config.yaml. -->
+  <link name="rslidar">
     <visual>
       <origin xyz="0.025 -0.0265 -0.025" rpy="${pi/2} 0 ${pi}"/>
@@ -140,8 +140,9 @@
     </visual>
   </link>
-  <joint name="livox_joint" type="fixed">
+  <!-- Legacy Livox joint name: livox_joint -->
+  <joint name="rslidar_joint" type="fixed">
     <origin xyz="$(arg xyz)" rpy="$(arg rpy)" />
     <parent link="base_link"/>
-    <child link="livox_frame"/>
+    <child link="rslidar"/>
   </joint>
 </robot>

File: My_nav/src/rm_nav_bringup/urdf/sentry_robot_sim.urdf (robot description, URDF)
Before this commit: robot sentry_robot, 8 links, 7 joints
Links:
- removed link livox_frame
- added link rslidar; visual mesh filename=model://mid360.stl scale=0.0008 0.0008 0.0008
Joints:
- removed joint livox_frame_joint
- added joint rslidar_joint: type fixed, parent base_link, child rslidar, origin xyz=0.12 0.0 0.175 rpy=0 0 0

File: My_nav/src/rm_nav_bringup/urdf/sentry_robot_sim.xacro (robot description, xacro)
@@ -11,5 +11,5 @@
     </inertial>
   </xacro:macro>
-  <!-- base_link to livox_frame -->
+  <!-- base_link to rslidar (legacy frame: livox_frame) -->
   <xacro:arg name="xyz" default="0.12 0.0 0.175" />
   <xacro:arg name="rpy" default="0 0 0" />
@@ -182,5 +182,5 @@
     <material>Gazebo/BuildingFrame</material>
   </gazebo>
-  <gazebo reference="livox_frame">
+  <gazebo reference="rslidar">
     <material>Gazebo/LightBlueLaser</material>
   </gazebo>
@@ -212,8 +212,8 @@
     </plugin>
   </gazebo>
-  <!-- mid360_imu plugin -->
+  <!-- Airy Lite IMU simulation -->
   <!-- https://github.com/ros-simulation/gazebo_ros_pkgs/wiki/ROS-2-Migration:-IMU-Sensors -->
   <gazebo reference="imu_link">
-    <sensor name="mid360_imu" type="imu">
+    <sensor name="airy_lite_imu" type="imu">
       <always_on>true</always_on>
       <update_rate>100</update_rate>
@@ -221,5 +221,6 @@
         <ros>
           <namespace>/</namespace>
-          <remapping>~/out:=/livox/imu</remapping>
+          <!-- Livox: ~/out:=/livox/imu -->
+          <remapping>~/out:=/rslidar_imu_data</remapping>
         </ros>
         <frame_name>imu_link</frame_name>
@@ -227,8 +228,8 @@
     </sensor>
   </gazebo>
-  <!-- Livox-Mid360  -->
-  <xacro:include filename="$(find ros2_livox_simulation)/urdf/mid360.xacro" />
-  <xacro:mid360 name="livox_frame" parent="base_link" topic="/livox/lidar">
+  <!-- Legacy Livox include/macro: ros2_livox_simulation, xacro:mid360 -->
+  <xacro:include filename="$(find robosense_sim_ros2)/urdf/airy_lite.xacro" />
+  <xacro:airy_lite name="rslidar" parent="base_link" topic="/rslidar_points">
     <origin xyz="$(arg xyz)" rpy="$(arg rpy)" />
-  </xacro:mid360>
+  </xacro:airy_lite>
 </robot>

Commit message: 完善gazebo仿真环境

File: My_nav/src/gazebo/pb_rm_simulation/urdf/simulation_waking_robot.xacro (robot description, xacro)
@@ -11,5 +11,5 @@
     </inertial>
   </xacro:macro>
-  <!-- base_link to rslidar (legacy frame: livox_frame) -->
+  <!-- Airy Lite mounting pose: fixed transform from base_link to rslidar -->
   <xacro:arg name="xyz" default="0.12 0.0 0.175" />
   <xacro:arg name="rpy" default="0 0 0" />

File: My_nav/src/gazebo/robosense_sim_ros2/urdf/airy_lite.xacro (robot description, xacro)
@@ -24,5 +24,5 @@
         <origin xyz="0.025 -0.0265 -0.025" rpy="${pi/2} 0 ${pi}"/>
         <geometry>
-          <mesh filename="model://mid360.stl" scale="0.0008 0.0008 0.0008"/>
+          <mesh filename="model://airy_lite.stl" scale="0.0008 0.0008 0.0008"/>
         </geometry>
       </visual>

File: My_nav/src/rm_nav_bringup/urdf/sentry_robot_real.xacro (robot description, xacro)
@@ -133,5 +133,5 @@
       <origin xyz="0.025 -0.0265 -0.025" rpy="${pi/2} 0 ${pi}"/>
       <geometry>
-        <mesh filename="package://pb_rm_simulation/meshes/mid360.stl" scale="0.001 0.001 0.001"/>
+        <mesh filename="package://pb_rm_simulation/meshes/airy_lite.stl" scale="0.001 0.001 0.001"/>
       </geometry>
       <material name="blue">

File: My_nav/src/rm_nav_bringup/urdf/sentry_robot_sim.urdf (robot description, URDF)
Before this commit: robot sentry_robot, 8 links, 7 joints
Links:
- link rslidar: geometry visual mesh filename=model://airy_lite.stl scale=0.0008 0.0008 0.0008
